Commit message: fix config

File: src/my_robot/urdf/my_robot.xacro (robot description, xacro)
@@ -41,4 +41,9 @@
         <parent link="chassis"/>
         <axis xyz="0 1 0" rpy="0 0 0"/>
+    </joint>
+    <joint name="camera_optical_joint" type="fixed">
+        <origin xyz="0 0 0" rpy="-1.5707 0 -1.5707"/>
+        <parent link="camera"/>
+        <child link="camera_link_optical"/>
     </joint>
     <link name='chassis'>
@@ -182,3 +187,5 @@
         </visual>
     </link>
+    <link name="camera_link_optical">
+    </link>
 </robot>
